Commit message: Added cylindrical body. NOTE: visual is a tiny cylinder, so we can see the blades. collision cylinder wraps around quadcopters

File: rotors_description/urdf/roller.xacro (robot description, xacro)
@@ -23,8 +23,8 @@
   <xacro:property name="mesh_file" value="package://rotors_description/meshes/hummingbird.dae" />
   <xacro:property name="mass" value="1.5" /> <!-- [kg] -->
-  <xacro:property name="body_width" value="0.15" /> <!-- [m] -->
-  <xacro:property name="body_height" value="0.15" /> <!-- [m] -->
+  <xacro:property name="r" value="0.25" /> <!-- [m] -->
+  <xacro:property name="L" value="0.5" /> <!-- [m] -->
   <xacro:property name="mass_rotor" value="0.005" /> <!-- [kg] -->
-  <xacro:property name="arm_length" value="0.215" /> <!-- [m] -->
+  <xacro:property name="arm_length" value="0.2" /> <!-- [m] -->
   <xacro:property name="rotor_offset_top" value="0.037" /> <!-- [m] -->
   <xacro:property name="radius_rotor" value="0.1" /> <!-- [m] -->
@@ -39,5 +39,7 @@
   <!-- Property Blocks -->
   <xacro:property name="body_inertia">
-    <inertia ixx="0.09375" ixy="0.0" ixz="0.0" iyy="0.03125" iyz="0.0" izz="0.03125" /> <!-- [kg m^2] [kg m^2] [kg m^2] [kg m^2] [kg m^2] [kg m^2] -->
+    <inertia ixx="${0.5*mass*(r*r) + 0.333333*mass*(L*L)}" ixy="0.0" ixz="0.0"
+      iyy="${0.5*mass*(r*r) + 0.333333*mass*(L*L)}" iyz="0.0"
+      izz="${mass * (r*r)}" />
   </xacro:property>
   <!-- inertia of a single rotor, assuming it is a cuboid. Height=3mm, width=15mm -->
@@ -46,16 +48,14 @@
   </xacro:property>
   <!-- Included URDF Files -->
-  <xacro:include filename="$(find rotors_description)/urdf/multirotor_base.xacro" />
-  <!-- Instantiate multirotor_base_macro once -->
-  <xacro:multirotor_base_macro
+  <xacro:include filename="$(find rotors_description)/urdf/shapeshifter.xacro" />
+  <!-- Instantiate shapeshifter_base_macro once -->
+  <xacro:shapeshifter_base_macro
     robot_namespace="${namespace}"
     mass="${mass}"
-    body_width="${body_width}"
-    body_height="${body_height}"
-    use_mesh_file="${use_mesh_file}"
-    mesh_file="${mesh_file}"
+    r="${r}"
+    L="${L}"
     >
     <xacro:insert_block name="body_inertia" />
-  </xacro:multirotor_base_macro>
+  </xacro:shapeshifter_base_macro>
   <!-- Instantiate rotors -->
   <xacro:vertical_rotor
@@ -77,5 +77,5 @@
     use_own_mesh="false"
     mesh="">
-    <origin xyz="${sin45*arm_length} -${sin45*arm_length} ${rotor_offset_top}" rpy="0 0 0" />
+    <origin xyz="${sin45*arm_length} -${sin45*arm_length} ${r + rotor_offset_top}" rpy="0 0 0" />
     <xacro:insert_block name="rotor_inertia" />
   </xacro:vertical_rotor>
@@ -98,5 +98,5 @@
     use_own_mesh="false"
     mesh="">
-    <origin xyz="${sin45*arm_length} ${sin45*arm_length} ${rotor_offset_top}" rpy="0 0 0" />
+    <origin xyz="${sin45*arm_length} ${sin45*arm_length} ${r + rotor_offset_top}" rpy="0 0 0" />
     <xacro:insert_block name="rotor_inertia" />
   </xacro:vertical_rotor>
@@ -118,5 +118,5 @@
     use_own_mesh="false"
     mesh="">
-    <origin xyz="-${sin45*arm_length} ${sin45*arm_length} ${rotor_offset_top}" rpy="0 0 0" />
+    <origin xyz="-${sin45*arm_length} ${sin45*arm_length} ${r + rotor_offset_top}" rpy="0 0 0" />
     <xacro:insert_block name="rotor_inertia" />
   </xacro:vertical_rotor>
@@ -138,5 +138,5 @@
     use_own_mesh="false"
     mesh="">
-    <origin xyz="-${sin45*arm_length} -${sin45*arm_length} ${rotor_offset_top}" rpy="0 0 0" />
+    <origin xyz="-${sin45*arm_length} -${sin45*arm_length} ${r + rotor_offset_top}" rpy="0 0 0" />
     <xacro:insert_block name="rotor_inertia" />
   </xacro:vertical_rotor>
@@ -160,5 +160,5 @@
     use_own_mesh="false"
     mesh="">
-    <origin xyz="${sin45*arm_length} -${sin45*arm_length} -${rotor_offset_top}" rpy="${pi} 0 0" />
+    <origin xyz="${sin45*arm_length} -${sin45*arm_length} ${r - rotor_offset_top}" rpy="${pi} 0 0" />
     <xacro:insert_block name="rotor_inertia" />
   </xacro:vertical_rotor>
@@ -181,5 +181,5 @@
     use_own_mesh="false"
     mesh="">
-    <origin xyz="${sin45*arm_length} ${sin45*arm_length} -${rotor_offset_top}" rpy="${pi} 0 0" />
+    <origin xyz="${sin45*arm_length} ${sin45*arm_length} ${r - rotor_offset_top}" rpy="${pi} 0 0" />
     <xacro:insert_block name="rotor_inertia" />
   </xacro:vertical_rotor>
@@ -201,5 +201,5 @@
     use_own_mesh="false"
     mesh="">
-    <origin xyz="-${sin45*arm_length} ${sin45*arm_length} -${rotor_offset_top}" rpy="${pi} 0 0" />
+    <origin xyz="-${sin45*arm_length} ${sin45*arm_length} ${r - rotor_offset_top}" rpy="${pi} 0 0" />
     <xacro:insert_block name="rotor_inertia" />
   </xacro:vertical_rotor>
@@ -221,5 +221,5 @@
     use_own_mesh="false"
     mesh="">
-    <origin xyz="-${sin45*arm_length} -${sin45*arm_length} -${rotor_offset_top}" rpy="${pi} 0 0" />
+    <origin xyz="-${sin45*arm_length} -${sin45*arm_length} ${r - rotor_offset_top}" rpy="${pi} 0 0" />
     <xacro:insert_block name="rotor_inertia" />
   </xacro:vertical_rotor>
